Commit message: feat(rl): spotmicro_v3.0 URDF 수정

File: ai_training/rl/legged_gym/resources/robots/spotmicro_test/urdf/spotmicro_test.urdf (robot description, URDF)
Before this commit: robot spot_micro, 23 links, 22 joints
Links:
- added link battery_link, mass 0.42; collision box size=0.13 0.045 0.035; visual box size=0.13 0.045 0.035
- link base_link: mass 1.2 -> 0.58
- link front_left_shoulder_link: mass 0.10 -> 0.09
- link front_link: mass 0.001 -> 0.285
- link front_right_shoulder_link: mass 0.10 -> 0.09
- link rear_left_shoulder_link: mass 0.10 -> 0.09
- link rear_link: mass 0.001 -> 0.1
- link rear_right_shoulder_link: mass 0.10 -> 0.09
Joints:
- added joint base_battery: type fixed, parent base_link, child battery_link

Commit message: v6.0 common IK train

File: ai_training/rl/legged_gym/resources/robots/spotmicro_test/urdf/spotmicro_test.urdf (robot description, URDF)
Before this commit: robot spot_micro, 24 links, 23 joints
Joints:
- joint front_left_foot: origin xyz=0.01 0 -0.12 rpy=0 0 0 -> xyz=0 0 -0.105 rpy=0 0 0
- joint front_left_toe: origin xyz=0 0 -0.115 -> xyz=0 0 -0.130
- joint front_right_foot: origin xyz=0.01 0 -0.12 rpy=0 0 0 -> xyz=0 0 -0.105 rpy=0 0 0
- joint front_right_toe: origin xyz=0 0 -0.115 -> xyz=0 0 -0.130
- joint rear_left_foot: origin xyz=0.01 0 -0.12 rpy=0 0 0 -> xyz=0 0 -0.105 rpy=0 0 0
- joint rear_left_toe: origin xyz=0 0 -0.115 -> xyz=0 0 -0.130
- joint rear_right_foot: origin xyz=0.01 0 -0.12 rpy=0 0 0 -> xyz=0 0 -0.105 rpy=0 0 0
- joint rear_right_toe: origin xyz=0 0 -0.115 -> xyz=0 0 -0.130

Commit message: fix: urdf toe change

File: ai_training/rl/legged_gym/resources/robots/spotmicro_test/urdf/spotmicro_test.urdf (robot description, URDF)
Before this commit: robot spot_micro, 24 links, 23 joints
Links:
- link front_left_toe_link: mass 0.015 -> 0.005; geometry collision sphere radius=0.015
- link front_right_toe_link: mass 0.015 -> 0.005; geometry collision sphere radius=0.015
- link rear_left_toe_link: mass 0.015 -> 0.005; geometry collision sphere radius=0.015
- link rear_right_toe_link: mass 0.015 -> 0.005; geometry collision sphere radius=0.015

Commit message: fix: urdf fix

File: ai_training/rl/legged_gym/resources/robots/spotmicro_test/urdf/spotmicro_test.urdf (robot description, URDF)
Before this commit: robot spot_micro, 24 links, 23 joints
Links:
- link front_left_toe_link: mass 0.015 -> 0.005; geometry collision sphere radius=0.015
- link front_right_toe_link: mass 0.015 -> 0.005; geometry collision sphere radius=0.015
- link rear_left_toe_link: mass 0.015 -> 0.005; geometry collision sphere radius=0.015
- link rear_right_toe_link: mass 0.015 -> 0.005; geometry collision sphere radius=0.015
Joints:
- joint front_left_foot: origin xyz=0 0 -0.105 rpy=0 0 0 -> xyz=0.01 0 -0.12 rpy=0 0 0
- joint front_left_toe: origin xyz=0 0 -0.130 -> xyz=0 0 -0.115
- joint front_right_foot: origin xyz=0 0 -0.105 rpy=0 0 0 -> xyz=0.01 0 -0.12 rpy=0 0 0
- joint front_right_toe: origin xyz=0 0 -0.130 -> xyz=0 0 -0.115
- joint rear_left_foot: origin xyz=0 0 -0.105 rpy=0 0 0 -> xyz=0.01 0 -0.12 rpy=0 0 0
- joint rear_left_toe: origin xyz=0 0 -0.130 -> xyz=0 0 -0.115
- joint rear_right_foot: origin xyz=0 0 -0.105 rpy=0 0 0 -> xyz=0.01 0 -0.12 rpy=0 0 0
- joint rear_right_toe: origin xyz=0 0 -0.130 -> xyz=0 0 -0.115
